File: CapiNetIO.kicad_sch (KiCad schematic)
At the start: 91 parts, among them J1 USB_B_Micro, J2 SWD Prg, J3 1963421, J4 USART3, J5 Conn_02x05_Counter_Clockwise, Q1 MMBT2222A, Q2 MMBT2222A, Q3 MMBT2222A, Q4 MMBT2222A, SW1 SW_SPDT, U1 STM32F446RETx, U3 AMS1117-3.3, Y1 16MHz

Commit message: Checked footprints and pcb constrains, time to start tracing
Parts:
- removed D6, D7: 5KPxxCA, Diode_THT:D_P600_R-6_P20.00mm_Horizontal, symbol Diode:5KPxxCA
- added D5, D6: ESD5Zxx, Diode_SMD:D_SOD-523, symbol Diode:ESD5Zxx
- C1, C10, C11, C14, C15, C2, C3, C4: footprint Capacitor_SMD:C_01005_0402Metric -> Capacitor_SMD:C_0603_1608Metric
- C6, C7, C8, C9: footprint Capacitor_SMD:C_0402_1005Metric -> Capacitor_SMD:C_0603_1608Metric
Connections:
- net 485A+: now also D5.1 (K)
- net 485B-: now also D6.1 (K)
- net GND: now also D5.2 (A), D6.2 (A)
Changed lines of the file:
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@@
 	)
 	(junction
-		(at 374.65 49.53)
-		(diameter 0)
-		(color 0 0 0 0)
-	)
-	(junction
 		(at 160.02 44.45)
 		(diameter 0)
@@
 	)
 	(junction
+		(at 374.65 49.53)
+		(diameter 0)
+		(color 0 0 0 0)
+	)
+	(junction
 		(at 360.68 168.91)
 		(diameter 0)
@@
 	)
 	(junction
+		(at 381 52.07)
+		(diameter 0)
+		(color 0 0 0 0)
+	)
+	(junction
 		(at 189.23 43.18)
 		(diameter 0)
@@
 		(color 0 0 0 0)
 	)
-	(junction
-		(at 381 52.07)
-		(diameter 0)
-		(color 0 0 0 0)
-	)
 	(no_connect
 		(at 209.55 115.57)
@@
 	(wire
 		(pts
+			(xy 374.65 49.53) (xy 383.54 49.53)
+		)
+		(stroke
+			(width 0)
+			(type default)
+		)
+	)
+	(wire
+		(pts
 			(xy 186.69 44.45) (xy 186.69 43.18)
 		)
@@
 	(wire
 		(pts
+			(xy 381 52.07) (xy 383.54 52.07)
+		)
+		(stroke
+			(width 0)
+			(type default)
+		)
+	)
+	(wire
+		(pts
 			(xy 162.56 193.04) (xy 147.32 193.04)
 		)
@@
 	(wire
 		(pts
-			(xy 381 52.07) (xy 383.54 52.07)
-		)
-		(stroke
-			(width 0)
-			(type default)
-		)
-	)
-	(wire
-		(pts
 			(xy 154.94 87.63) (xy 168.91 87.63)
 		)
@@
 	(wire
 		(pts
-			(xy 374.65 49.53) (xy 383.54 49.53)
-		)
-		(stroke
-			(width 0)
-			(type default)
-		)
-	)
-	(wire
-		(pts
 			(xy 284.48 90.17) (xy 288.29 90.17)
 		)
@@
 			)
 		)
-		(property "Footprint" "Capacitor_SMD:C_0402_1005Metric"
+		(property "Footprint" "Capacitor_SMD:C_0603_1608Metric"
 			(at 219.4052 43.18 0)
 			(effects
@@
 	)
 	(symbol
-		(lib_id "Diode:5KPxxCA")
-		(at 374.65 53.34 90)
-		(unit 1)
-		(exclude_from_sim no)
-		(in_bom yes)
-		(on_board yes)
-		(dnp no)
-		(fields_autoplaced yes)
-		(property "Reference" "D6"
-			(at 377.19 52.0699 90)
-			(effects
-				(font
-					(size 1.27 1.27)
-				)
-				(justify right)
-			)
-		)
-		(property "Value" "5KPxxCA"
-			(at 377.19 54.6099 90)
-			(effects
-				(font
-					(size 1.27 1.27)
-				)
-				(justify right)
-			)
-		)
-		(property "Footprint" "Diode_THT:D_P600_R-6_P20.00mm_Horizontal"
-			(at 379.73 53.34 0)
-			(effects
-				(font
-					(size 1.27 1.27)
-				)
-				(hide yes)
-			)
-		)
-		(property "Datasheet" "https://diotec.com/tl_files/diotec/files/pdf/datasheets/5kp65.pdf"
-			(at 374.65 53.34 0)
-			(effects
-				(font
-					(size 1.27 1.27)
-				)
-				(hide yes)
-			)
-		)
-		(property "Description" "5000W bidirectional Transient Voltage Suppressor, P-600"
-			(at 374.65 53.34 0)
-			(effects
-				(font
-					(size 1.27 1.27)
-				)
-				(hide yes)
-			)
-		)
-		(pin "2"
-		)
-		(pin "1"
-		)
-		(instances
-			(project ""
-				(path "/1a5652bf-ba49-4248-8cd9-02a29183ef4e"
-					(reference "D6")
-					(unit 1)
-				)
-			)
-		)
-	)
-	(symbol
 		(lib_id "Device:R")
 		(at 234.95 193.04 90)
@@
 			)
 		)
-		(property "Footprint" "Capacitor_SMD:C_01005_0402Metric"
+		(property "Footprint" "Capacitor_SMD:C_0603_1608Metric"
 			(at 147.0152 43.18 0)
 			(effects
@@
 			)
 		)
-		(property "Footprint" "Capacitor_SMD:C_0402_1005Metric"
+		(property "Footprint" "Capacitor_SMD:C_0603_1608Metric"
 			(at 100.0252 59.69 0)
 			(effects
@@
 			)
 		)
-		(property "Footprint" "Capacitor_SMD:C_0402_1005Metric"
+		(property "Footprint" "Capacitor_SMD:C_0603_1608Metric"
 			(at 233.3752 43.18 0)
 			(effects
@@
 			)
 		)
-		(property "Footprint" "Capacitor_SMD:C_01005_0402Metric"
+		(property "Footprint" "Capacitor_SMD:C_0603_1608Metric"
 			(at 101.2952 93.98 0)
 			(effects
@@
 			)
 		)
-		(property "Footprint" "Capacitor_SMD:C_01005_0402Metric"
+		(property "Footprint" "Capacitor_SMD:C_0603_1608Metric"
 			(at 160.9852 43.18 0)
 			(effects
@@
 			)
 		)
-		(property "Footprint" "Capacitor_SMD:C_01005_0402Metric"
+		(property "Footprint" "Capacitor_SMD:C_0603_1608Metric"
 			(at 371.8052 43.18 0)
 			(effects
@@
 			)
 		)
-		(property "Footprint" "Capacitor_SMD:C_01005_0402Metric"
+		(property "Footprint" "Capacitor_SMD:C_0603_1608Metric"
 			(at 135.5852 93.98 0)
 			(effects
@@
 	)
 	(symbol
+		(lib_id "Diode:ESD5Zxx")
+		(at 381 55.88 270)
+		(unit 1)
+		(exclude_from_sim no)
+		(in_bom yes)
+		(on_board yes)
+		(dnp no)
+		(fields_autoplaced yes)
+		(property "Reference" "D5"
+			(at 383.54 54.6099 90)
+			(effects
+				(font
+					(size 1.27 1.27)
+				)
+				(justify left)
+			)
+		)
+		(property "Value" "ESD5Zxx"
+			(at 383.54 57.1499 90)
+			(effects
+				(font
+					(size 1.27 1.27)
+				)
+				(justify left)
+			)
+		)
+		(property "Footprint" "Diode_SMD:D_SOD-523"
+			(at 376.555 55.88 0)
+			(effects
+				(font
+					(size 1.27 1.27)
+				)
+				(hide yes)
+			)
+		)
+		(property "Datasheet" "https://www.onsemi.com/pdf/datasheet/esd5z2.5t1-d.pdf"
+			(at 381 55.88 0)
+			(effects
+				(font
+					(size 1.27 1.27)
+				)
+				(hide yes)
+			)
+		)
+		(property "Description" "ESD Protection Diode, SOD-523"
+			(at 381 55.88 0)
+			(effects
+				(font
+					(size 1.27 1.27)
+				)
+				(hide yes)
+			)
+		)
+		(pin "2"
+		)
+		(pin "1"
+		)
+		(instances
+			(project ""
+				(path "/1a5652bf-ba49-4248-8cd9-02a29183ef4e"
+					(reference "D5")
+					(unit 1)
+				)
+			)
+		)
+	)
+	(symbol
 		(lib_id "power:GND")
 		(at 218.44 44.45 0)
@@
 	)
 	(symbol
+		(lib_id "Diode:ESD5Zxx")
+		(at 374.65 53.34 270)
+		(unit 1)
+		(exclude_from_sim no)
+		(in_bom yes)
+		(on_board yes)
+		(dnp no)
+		(fields_autoplaced yes)
+		(property "Reference" "D6"
+			(at 377.19 52.0699 90)
+			(effects
+				(font
+					(size 1.27 1.27)
+				)
+				(justify left)
+			)
+		)
+		(property "Value" "ESD5Zxx"
+			(at 377.19 54.6099 90)
+			(effects
+				(font
+					(size 1.27 1.27)
+				)
+				(justify left)
+			)
+		)
+		(property "Footprint" "Diode_SMD:D_SOD-523"
+			(at 370.205 53.34 0)
+			(effects
+				(font
+					(size 1.27 1.27)
+				)
+				(hide yes)
+			)
+		)
+		(property "Datasheet" "https://www.onsemi.com/pdf/datasheet/esd5z2.5t1-d.pdf"
+			(at 374.65 53.34 0)
+			(effects
+				(font
+					(size 1.27 1.27)
+				)
+				(hide yes)
+			)
+		)
+		(property "Description" "ESD Protection Diode, SOD-523"
+			(at 374.65 53.34 0)
+			(effects
+				(font
+					(size 1.27 1.27)
+				)
+				(hide yes)
+			)
+		)
+		(pin "2"
+		)
+		(pin "1"
+		)
+		(instances
+			(project "CapiNetIO"
+				(path "/1a5652bf-ba49-4248-8cd9-02a29183ef4e"
+					(reference "D6")
+					(unit 1)
+				)
+			)
+		)
+	)
+	(symbol
 		(lib_id "power:+3.3V")
 		(at 363.22 35.56 0)
@@
 			)
 		)
-		(property "Footprint" "Capacitor_SMD:C_0402_1005Metric"
+		(property "Footprint" "Capacitor_SMD:C_0603_1608Metric"
 			(at 256.2352 41.91 0)
 			(effects
@@
 			)
 		)
-		(property "Footprint" "Capacitor_SMD:C_01005_0402Metric"
+		(property "Footprint" "Capacitor_SMD:C_0603_1608Metric"
 			(at 173.6852 43.18 0)
 			(effects
@@
 	)
 	(symbol
-		(lib_id "Diode:5KPxxCA")
-		(at 381 55.88 90)
-		(unit 1)
-		(exclude_from_sim no)
-		(in_bom yes)
-		(on_board yes)
-		(dnp no)
-		(fields_autoplaced yes)
-		(property "Reference" "D7"
-			(at 383.54 54.6099 90)
-			(effects
-				(font
-					(size 1.27 1.27)
-				)
-				(justify right)
-			)
-		)
-		(property "Value" "5KPxxCA"
-			(at 383.54 57.1499 90)
-			(effects
-				(font
-					(size 1.27 1.27)
-				)
-				(justify right)
-			)
-		)
-		(property "Footprint" "Diode_THT:D_P600_R-6_P20.00mm_Horizontal"
-			(at 386.08 55.88 0)
-			(effects
-				(font
-					(size 1.27 1.27)
-				)
-				(hide yes)
-			)
-		)
-		(property "Datasheet" "https://diotec.com/tl_files/diotec/files/pdf/datasheets/5kp65.pdf"
-			(at 381 55.88 0)
-			(effects
-				(font
-					(size 1.27 1.27)
-				)
-				(hide yes)
-			)
-		)
-		(property "Description" "5000W bidirectional Transient Voltage Suppressor, P-600"
-			(at 381 55.88 0)
-			(effects
-				(font
-					(size 1.27 1.27)
-				)
-				(hide yes)
-			)
-		)
-		(pin "2"
-		)
-		(pin "1"
-		)
-		(instances
-			(project "CapiNetIO"
-				(path "/1a5652bf-ba49-4248-8cd9-02a29183ef4e"
-					(reference "D7")
-					(unit 1)
-				)
-			)
-		)
-	)
-	(symbol
 		(lib_id "Device:R")
 		(at 384.81 73.66 90)
@@
 			)
 		)
-		(property "Footprint" "Capacitor_SMD:C_01005_0402Metric"
+		(property "Footprint" "Capacitor_SMD:C_0603_1608Metric"
 			(at 133.0452 43.18 0)
 			(effects
@@
 			)
 		)
-		(property "Footprint" "Capacitor_SMD:C_01005_0402Metric"
+		(property "Footprint" "Capacitor_SMD:C_0603_1608Metric"
 			(at 310.8452 43.18 0)
 			(effects

Commit message: Changed pins GPIO_Out0-3 and GPIO_In0-3 to a more accessible ones. Added project CubeMX
Parts:
- renumbered J3 to Ext_PWR1, JP1 to JmpPWR1, LED_Outputs2 to LED_Inputs1, J2 to SWD_PRG1, J4 to USART3
Connections:
- net GPIO_INCon4 is gone; now on net GPIO_in3: OptoIn1.10, R_48.1
- net GPIO_INCon0: now also R15.2; no longer OptoIn1.16, R_45.1
- net GPIO_INCon1: now also R16.2, U1.34 (PB13); no longer OptoIn1.14, R_46.1
- net GPIO_INCon2: now also R17.2, U1.35 (PB14); no longer OptoIn1.12, R_47.1, U1.34 (PB13)
- net GPIO_INCon3: now also R18.2; no longer U1.35 (PB14)
- net GPIO_in0: now also OptoIn1.16, R_45.1; no longer R15.2
- net GPIO_in1: now also OptoIn1.14, R_46.1; no longer R16.2
- net GPIO_in2: now also OptoIn1.12, R_47.1; no longer R17.2
- net GPIO_in3: no longer R18.2
- net GPIO_out0: now also U1.28 (PB2); no longer U1.55 (PB3)
- net GPIO_out1: now also U1.24 (PC4); no longer U1.56 (PB4)
- net GPIO_out2: now also U1.26 (PB0); no longer U1.57 (PB5)
- net GPIO_out3: now also U1.27 (PB1); no longer U1.58 (PB6)
- net Config3: now reaches Configuration1.5 (NO_1), R18.1
- net Config2: now reaches Configuration1.6 (NO_2), R17.1
- net Config1: now reaches Configuration1.7 (NO_3), R16.1
- net Config0: now reaches Configuration1.8 (NO_4), R15.1
Other:
- moved on the sheet: Configuration1, R15, R16, R17, R18
