File: CapiNetIO.kicad_sch (KiCad schematic)
At the start: 91 parts, among them J1 USB_B_Micro, J5 Conn_02x05_Counter_Clockwise, Q1 MMBT2222A, Q2 MMBT2222A, Q3 MMBT2222A, Q4 MMBT2222A, SW1 SW_SPDT, U1 STM32F446RETx, U3 AMS1117-3.3, Y1 16MHz

Commit message: working on the pcb side, tidying up io
Parts:
- added C16: 100n, Capacitor_SMD:C_0603_1608Metric, symbol Device:C
- renumbered R_31 to R31, R_35 to R35, R_36 to R36, R_37 to R37, R_38 to R38
Connections:
- net +3.3V: now also C16.1
- net Config0: now also Configuration1.5 (NO_1); no longer Configuration1.8 (NO_4)
- net Config1: now also Configuration1.6 (NO_2); no longer Configuration1.7 (NO_3)
- net Config2: now also Configuration1.7 (NO_3); no longer Configuration1.6 (NO_2)
- net Config3: now also Configuration1.8 (NO_4); no longer Configuration1.5 (NO_1)
- net GND: now also C16.2
- net at D2.1 (K): now also R_42.1; no longer Inputs1.3
- net at D2.2 (A): now also Inputs1.3; no longer R_42.1
- net at R_43.1: now also D3.1 (K); no longer D3.2 (A)
- net at Inputs1.2: now also D1.2 (A); no longer D1.1 (K)
- net at Inputs1.4: now also D3.2 (A); no longer D3.1 (K)
- net at Inputs1.5: now also D4.2 (A); no longer D4.1 (K)
- net at R_41.1: now also D1.1 (K); no longer D1.2 (A)
- net at R_44.1: now also D4.1 (K); no longer D4.2 (A)
Other:
- moved on the sheet: Configuration1, D1, R15, R16, R17, R18
